Commit message: New urdf and parser

File: src/mike_description/urdf/mike.urdf (robot description, URDF)
Before this commit: robot Mike, 0 links, 0 joints
Links:
- added link base_link; visual box size=0.34925 0.34925 0.1016
- added link camera_link; visual box size=0.0762 0.2794 0.0762
- added link front__wheel; visual cylinder length=.04 radius=0.0381
- added link front_wheel_holder; visual box size=0.0381 .0381 .05
- added link kinect_holder; visual box size=0.127 .3302 .1778
- added link left_leg; visual box size=0.0254 .0254 .06
- added link left_wheel; visual cylinder length=.0254 radius=0.0762
- added link neck; visual box size=1.143 .0889 .0889
- added link right__wheel; visual cylinder length=.0254 radius=0.0762
- added link right_leg; visual box size=0.0254 .0254 .06
Joints:
- added joint base_to_front_wheel_holder: type fixed, parent base_link, child front_wheel_holder, origin xyz=0 -0.127 -0.0635 rpy=0 0 0
- added joint base_to_left_leg: type fixed, parent base_link, child left_leg, origin xyz=-0.1905 0.127 -0.0762 rpy=0 1.57075 0
- added joint base_to_neck: type fixed, parent base_link, child neck, origin xyz=0 0 -0.0508
- added joint base_to_right_leg: type fixed, parent base_link, child right_leg, origin xyz=0.1905 0.127 -0.0762 rpy=0 1.57075 0
- added joint front__wheel_joint: type continuous, parent front_wheel_holder, child front__wheel, origin xyz=0 0 -0.0508 rpy=0 1.57075 0, axis 0 0 1, limit effort=100 velocity=10
- added joint kinect_holder_holder_to_camera_link: type fixed, parent kinect_holder, child camera_link, origin xyz=0 0 1.3081 rpy=0 0 1.57075
- added joint left_wheel_to_left_leg: type continuous, parent left_leg, child left_wheel, origin xyz=0 0.0 0 rpy=0 0 0, limit effort=100 velocity=10
- added joint neck_to_kinect_holder_holder: type fixed, parent neck, child kinect_holder
- added joint right__wheel_joint: type continuous, parent right_leg, child right__wheel, origin xyz=0 0 0 rpy=0 0 0, axis 0 0 1, limit effort=100 velocity=10

Commit message: add temp Kinectodom

File: src/mike_description/urdf/mike.urdf (robot description, URDF)
Before this commit: robot Mike, 10 links, 9 joints
Links:
- added link odom; visual box size=0.0762 0.2794 0.0762
Joints:
- added joint odom_to_camera_link: type fixed, parent camera_link, child odom

Commit message: differential_drive

File: src/mike_description/urdf/mike.urdf (robot description, URDF)
Before this commit: robot Mike, 11 links, 10 joints
Links:
- removed link odom
Joints:
- removed joint odom_to_camera_link

Commit message: gmapping

File: src/mike_description/urdf/mike.urdf (robot description, URDF)
Before this commit: robot Mike, 10 links, 9 joints
Joints:
- joint kinect_holder_holder_to_camera_link: origin xyz=0 0 1.3081 rpy=0 0 1.57075 -> xyz=0 0 1.3081 rpy=0 0 0

Commit message: playing with the odometry for mapping

File: src/mike_description/urdf/mike.urdf (robot description, URDF)
Before this commit: robot Mike, 10 links, 9 joints
Links:
- removed link front__wheel
- removed link front_wheel_holder
- removed link kinect_holder
- removed link left_leg
- removed link left_wheel
- removed link neck
- removed link right__wheel
- removed link right_leg
- link base_link: geometry visual box size=0.3048 0.3048 0.2667
Joints:
- removed joint base_to_front_wheel_holder
- removed joint base_to_left_leg
- removed joint base_to_neck
- removed joint base_to_right_leg
- removed joint front__wheel_joint
- removed joint kinect_holder_holder_to_camera_link
- removed joint left_wheel_to_left_leg
- removed joint neck_to_kinect_holder_holder
- removed joint right__wheel_joint
- added joint base_link_holder_to_camera_link: type fixed, parent base_link, child camera_link, origin xyz=0.1143 0 0.19685 rpy=0 0 0
